Commit message: add gazebo, update readme

File: src/bot_description/urdf/xacro/robot.urdf.xacro (robot description, xacro)
@@ -1,3 +1,4 @@
-<robot xmlns:xacro="http://www.ros.org/wiki/xacro" name="robot">
+<robot xmlns:xacro="http://www.ros.org/wiki/xacro" name="III-Robot">
+    <xacro:include filename="calc_inertia.urdf.xacro"/>
     <xacro:include filename="robot_base.urdf.xacro"/>
     <xacro:include filename="robot_laser.urdf.xacro"/>

File: src/bot_description/urdf/xacro/robot_base.urdf.xacro (robot description, xacro)
@@ -31,4 +31,10 @@
             </geometry>
         </visual>
+        <collision>
+            <geometry>
+                <sphere radius="0.001"/>
+            </geometry>
+        </collision>
+        <xacro:sphere_inertial_matrix mass="0.001" radius="0.001" />
     </link>
     <!-- 3 set base_link -->
@@ -40,4 +46,10 @@
             <material name="white"/>
         </visual>
+        <collision>
+            <geometry>
+                <box size="${CAR_LENGTH} ${CAR_WIDTH} ${CAR_HEIGHT}"/>
+            </geometry>
+        </collision>
+        <xacro:box_inertial_matrix mass="5" length="${CAR_LENGTH}" width="${CAR_WIDTH}" height="${CAR_HEIGHT}" />
     </link>
     <!-- 4 connect base_footprint with base_link -->
@@ -48,4 +60,7 @@
         <origin xyz="0.0 0.0 ${CAR_HEIGHT/2+DISTANCE}"/>
     </joint>
+    <gazebo reference="base_link">
+        <material>Gazebo/White</material>
+    </gazebo>
     <!-- 5 定义车轮相关的宏 -->
     <!-- 宏函数创建规则：
@@ -62,5 +77,15 @@
                 <origin rpy="${PI/2} 0.0 0.0"/>
             </visual>
+            <collision>
+                <geometry>
+                    <cylinder radius="${WHEEL_RADIUS}" length="${WHEEL_LEHGTH}"/>
+                </geometry>
+                <origin rpy="${PI/2} 0.0 0.0"/>
+            </collision>
+            <xacro:cylinder_inertial_matrix mass="1" radius="${WHEEL_RADIUS}" length="${WHEEL_LEHGTH}" />
         </link>
+        <gazebo reference="${link_name}">
+            <material>Gazebo/Black</material>
+        </gazebo>
         <joint name="${link_name}2base_link" type="continuous">
             <parent link="base_link"/>
@@ -79,5 +104,15 @@
                 <origin rpy="${PI/2} 0.0 0.0"/>
             </visual>
+            <collision>
+                <geometry>
+                    <cylinder radius="0.01" length="${WHEEL_CAR_DISTANCE}"/>
+                </geometry>
+                <origin rpy="${PI/2} 0.0 0.0"/>
+            </collision>
+            <xacro:cylinder_inertial_matrix mass="1" radius="0.01" length="${WHEEL_CAR_DISTANCE}" />
         </link>
+        <gazebo reference="${link_name}_link">
+            <material>Gazebo/Black</material>
+        </gazebo>
         <joint name="${link_name}_joint" type="fixed">
             <parent link="base_link"/>
@@ -93,5 +128,15 @@
                 <origin rpy="0.0 0.0 0.0"/>
             </visual>
+            <collision>
+                <geometry>
+                    <box size="0.01 0.01 0.16"/>
+                </geometry>
+                <origin rpy="0.0 0.0 0.0"/>
+            </collision>
+            <xacro:box_inertial_matrix mass="1" length="0.01" width="0.01" height="0.16" />
         </link>
+        <gazebo reference="${link_name}_pillar">
+            <material>Gazebo/Black</material>
+        </gazebo>
         <joint name="${link_name}_pillar2base_joint" type="fixed">
             <parent link="base_link"/>
@@ -112,5 +157,14 @@
             <material name="white"/>
         </visual>
+        <collision>
+            <geometry>
+                <box size="${CAR_LENGTH} ${CAR_WIDTH} 0.005"/>
+            </geometry>
+        </collision>
+        <xacro:box_inertial_matrix mass="1" length="${CAR_LENGTH}" width="${CAR_WIDTH}" height="0.005" />
     </link>
+    <gazebo reference="base_link_2">
+        <material>Gazebo/White</material>
+    </gazebo>
     <joint name="base_link2base_link_2" type="fixed">
         <parent link="base_link"/>

File: src/bot_description/urdf/xacro/robot_camera.urdf.xacro (robot description, xacro)
@@ -2,5 +2,5 @@
     <xacro:property name="CAMERA_RADIUS" value="0.07" />
     <xacro:property name="FOOTHOLD_RADIUS" value="0.111" />
-    <xacro:property name="FOOTHOLD_HEIGHT" value="0.005" />
+    <xacro:property name="FOOTHOLD_HEIGHT" value="0.01" />
     <link name="foothold_base_1">
         <visual>
@@ -10,4 +10,10 @@
             <material name="black" />
         </visual>
+        <collision>
+            <geometry>
+                <cylinder radius="${FOOTHOLD_RADIUS}" length="${FOOTHOLD_HEIGHT}"/>
+            </geometry>
+        </collision>
+        <xacro:cylinder_inertial_matrix mass="0.5" radius="${FOOTHOLD_RADIUS}" length="${FOOTHOLD_HEIGHT}"/>
     </link>
     <joint name="foothold_base1_2_base_link2" type="fixed">
@@ -23,4 +29,10 @@
             <material name="black" />
         </visual>
+        <collision>
+            <geometry>
+                <box size="${FOOTHOLD_HEIGHT} 0.05 0.23"/>
+            </geometry>
+        </collision>
+        <xacro:box_inertial_matrix mass="0.1" length="${FOOTHOLD_HEIGHT}" width="0.05" height="0.23"/>
     </link>
     <joint name="foothold_base12_joint" type="fixed">
@@ -36,4 +48,10 @@
             <material name="black" />
         </visual>
+        <collision>
+            <geometry>
+                <box size="0.06 0.05 ${FOOTHOLD_HEIGHT}"/>
+            </geometry>
+        </collision>
+        <xacro:box_inertial_matrix mass="0.1" length="0.06" width="0.05" height="${FOOTHOLD_HEIGHT}"/>
     </link>
     <joint name="foothold_base23_joint" type="fixed">
@@ -49,4 +67,10 @@
             <material name="black" />
         </visual>
+        <collision>
+            <geometry>
+                <cylinder radius="0.07" length="${FOOTHOLD_HEIGHT}"/>
+            </geometry>
+        </collision>
+        <xacro:cylinder_inertial_matrix mass="0.1" radius="0.07" length="${FOOTHOLD_HEIGHT}"/>
     </link>
     <joint name="foothold_base34_joint" type="fixed">
@@ -62,4 +86,10 @@
             <material name="white" />
         </visual>
+        <collision>
+            <geometry>
+                <cylinder radius="0.02" length="0.07"/>
+            </geometry>
+        </collision>
+        <xacro:cylinder_inertial_matrix mass="0.1" radius="0.02" length="0.007"/>
     </link>
     <joint name="camera_link2foothold4" type="continuous">
@@ -76,4 +106,10 @@
             <material name="white"/>
         </visual>
+        <collision>
+            <geometry>
+                <sphere radius="${CAMERA_RADIUS}"/>
+            </geometry>
+        </collision>
+        <xacro:sphere_inertial_matrix mass="5" radius="${CAMERA_RADIUS}" />
     </link>
     <joint name="camera_link2camera" type="fixed">
@@ -82,3 +118,21 @@
         <origin xyz="0.0 0.0 ${-(CAMERA_RADIUS+0.035)}"/>
     </joint>
+    <gazebo reference="foothold_base_1">
+        <material>Gazebo/Black</material>
+    </gazebo>
+    <gazebo reference="foothold_base_2">
+        <material>Gazebo/Black</material>
+    </gazebo>
+    <gazebo reference="foothold_base_3">
+        <material>Gazebo/Black</material>
+    </gazebo>
+    <gazebo reference="foothold_base_4">
+        <material>Gazebo/Black</material>
+    </gazebo>
+    <gazebo reference="camera_link">
+        <material>Gazebo/White</material>
+    </gazebo>
+    <gazebo reference="camera">
+        <material>Gazebo/White</material>
+    </gazebo>
 </robot>
