Commit message: update readme 1927

File: src/bot_description/urdf/bot_gazebo.xacro (robot description, xacro)
@@ -163,15 +163,14 @@
     <!-- motor -->
     <gazebo reference="front_left_motor">
-        <material>Gazebo/FlatBlack</material>
+        <material>Gazebo/Black</material>
     </gazebo>
     <gazebo reference="front_right_motor">
-        <material>Gazebo/FlatBlack</material>
+        <material>Gazebo/Black</material>
     </gazebo>
     <gazebo reference="back_left_motor">
-        <material>Gazebo/FlatBlack</material>
+        <material>Gazebo/Black</material>
     </gazebo>
     <gazebo reference="back_right_motor">
-        <material>Gazebo/FlatBlack</material>
+        <material>Gazebo/Black</material>
     </gazebo>
-    <!-- roller -->
 </robot>
