Commit message: add roller

File: src/bot_description/urdf/bot.urdf.xacro (robot description, xacro)
@@ -1,4 +1,5 @@
 <robot xmlns:xacro="http://www.ros.org/wiki/xacro" name="bot">
     <xacro:include filename="inertia.urdf.xacro"/>
+    <xacro:include filename="mecanum_wheel.xacro"/>
     <xacro:include filename="bot_base.urdf.xacro"/>
     <xacro:include filename="bot_gazebo.urdf.xacro"/>

File: src/bot_description/urdf/bot_base.urdf.xacro (robot description, xacro)
@@ -1,6 +1,6 @@
 <robot xmlns:xacro="http://www.ros.org/wiki/xacro">
-    <!-- 需要声明变量 -->
+    <!-- variable declaration -->
     <xacro:property name="PI" value="3.141592653" />
-    <!-- 离地间距 -->
+    <!-- Define the distance between the chassis and the ground -->
     <xacro:property name="z_offset" value="0.037" />
     <!-- color define -->
@@ -14,5 +14,5 @@
         <color rgba="0.8 0.0 0.0 0.7"/>
     </material>
-    <!-- 底盘参数 -->
+    <!-- chassis parameters -->
     <xacro:property name="bot_length" value="0.387" />
     <xacro:property name="bot_width" value="0.238" />
@@ -39,5 +39,5 @@
     <xacro:property name="motor_length" value="0.12" />
     <xacro:property name="motor_mass" value="0.3" />
-    <!-- 定义三个底盘  base_link_1 base_link_2 base_link_3-->
+    <!--   Define three chassis base_link_1 base_link_2 base_link_3-->
     <link name="base_link_1">
         <visual>
@@ -94,8 +94,9 @@
         <origin xyz="0.0 0.0 ${pillar_height_2+bot_height}"/>
     </joint>
+<!-- ************************************************************************************************************************************* -->
     <!-- wheel -->
-    <xacro:macro name="wheel_func" params="link_name front_flag left_flag">
+    <xacro:macro name="wheel_func" params="link_name front_flag left_flag angle">
         <!-- wheel -->
-        <link name="${link_name}">
+        <!-- <link name="${link_name}">
             <visual>
                 <geometry>
@@ -118,4 +119,12 @@
             <origin xyz="${wheel_joint_x * front_flag} ${wheel_joint_y * left_flag} ${wheel_joint_z}"/>
             <axis xyz="0 1 0"/>
+        </joint> -->
+        <xacro:property name="roller_angle" value="${PI/4}" />
+        <xacro:mecanum_wheel name="${link_name}" roller_angle = "${angle*roller_angle}"/>
+        <joint name="${link_name}_joint" type="continuous">
+            <parent link="base_link_1"/>
+            <child link="${link_name}"/>
+            <origin xyz="${wheel_joint_x * front_flag} ${wheel_joint_y * left_flag} ${wheel_joint_z}" rpy="${3*pi/2} 0 0"/>
+            <axis xyz="0 0 1"/>
         </joint>
         <!-- pillar -->
@@ -182,7 +191,7 @@
         </joint>
     </xacro:macro>
-    <xacro:wheel_func link_name="front_left" front_flag="1" left_flag="1"/>
-    <xacro:wheel_func link_name="front_right" front_flag="1" left_flag="-1"/>
-    <xacro:wheel_func link_name="back_left" front_flag="-1" left_flag="1"/>
-    <xacro:wheel_func link_name="back_right" front_flag="-1" left_flag="-1"/>
+    <xacro:wheel_func link_name="front_left" front_flag="1" left_flag="1" angle="-1"/>
+    <xacro:wheel_func link_name="front_right" front_flag="1" left_flag="-1 " angle="1"/>
+    <xacro:wheel_func link_name="back_left" front_flag="-1" left_flag="1" angle="1"/>
+    <xacro:wheel_func link_name="back_right" front_flag="-1" left_flag="-1" angle="-1"/>
 </robot>

File: src/bot_description/urdf/bot_gazebo.urdf.xacro (robot description, xacro)
@@ -13,14 +13,14 @@
     <!-- wheel -->
     <gazebo reference="front_left">
-        <material>Gazebo/Black</material>
+        <material>Gazebo/White</material>
     </gazebo>
     <gazebo reference="front_right">
-        <material>Gazebo/Black</material>
+        <material>Gazebo/White</material>
     </gazebo>
     <gazebo reference="back_left">
-        <material>Gazebo/Black</material>
+        <material>Gazebo/White</material>
     </gazebo>
     <gazebo reference="back_right">
-        <material>Gazebo/Black</material>
+        <material>Gazebo/White</material>
     </gazebo>
     <!-- pillar -->
@@ -62,3 +62,46 @@
         <material>Gazebo/FlatBlack</material>
     </gazebo>
+    <!-- roller -->
+    <xacro:macro name="gazebo_roller_color" params="link_name">
+        <gazebo reference="${link_name}_roller_1">
+            <material>Gazebo/Black</material>
+        </gazebo>
+        <gazebo reference="${link_name}_roller_2">
+            <material>Gazebo/Black</material>
+        </gazebo>
+        <gazebo reference="${link_name}_roller_3">
+            <material>Gazebo/Black</material>
+        </gazebo>
+        <gazebo reference="${link_name}_roller_4">
+            <material>Gazebo/Black</material>
+        </gazebo>
+        <gazebo reference="${link_name}_roller_5">
+            <material>Gazebo/Black</material>
+        </gazebo>
+        <gazebo reference="${link_name}_roller_6">
+            <material>Gazebo/Black</material>
+        </gazebo>
+        <gazebo reference="${link_name}_roller_7">
+            <material>Gazebo/Black</material>
+        </gazebo>
+        <gazebo reference="${link_name}_roller_8">
+            <material>Gazebo/Black</material>
+        </gazebo>
+        <gazebo reference="${link_name}_roller_9">
+            <material>Gazebo/Black</material>
+        </gazebo>
+        <gazebo reference="${link_name}_roller_10">
+            <material>Gazebo/Black</material>
+        </gazebo>
+        <gazebo reference="${link_name}_roller_11">
+            <material>Gazebo/Black</material>
+        </gazebo>
+        <gazebo reference="${link_name}_roller_12">
+            <material>Gazebo/Black</material>
+        </gazebo>
+    </xacro:macro>
+    <xacro:gazebo_roller_color link_name="front_left"/>
+    <xacro:gazebo_roller_color link_name="front_right"/>
+    <xacro:gazebo_roller_color link_name="back_left"/>
+    <xacro:gazebo_roller_color link_name="back_right"/>
 </robot>

Commit message: add lidar plugin

File: src/bot_description/urdf/bot.urdf.xacro (robot description, xacro)
@@ -1,6 +1,8 @@
 <robot xmlns:xacro="http://www.ros.org/wiki/xacro" name="bot">
     <xacro:include filename="inertia.urdf.xacro"/>
+    <xacro:include filename="material.urdf.xacro"/>
     <xacro:include filename="bot_wheel.urdf.xacro"/>
     <xacro:include filename="bot_base.urdf.xacro"/>
+    <xacro:include filename="bot_lidar.urdf.xacro"/>
     <xacro:include filename="bot_gazebo.xacro"/>
     <xacro:include filename="bot_gazebo_plugin.xacro"/>

File: src/bot_description/urdf/bot_base.urdf.xacro (robot description, xacro)
@@ -4,14 +4,4 @@
     <!-- Define the distance between the chassis and the ground -->
     <xacro:property name="z_offset" value="0.037" />
-    <!-- color define -->
-    <material name="white">
-        <color rgba="0.7 0.7 0.7 0.8"/>
-    </material>
-    <material name="black">
-        <color rgba="0.2 0.2 0.2 0.7"/>
-    </material>
-    <material name="red">
-        <color rgba="0.8 0.0 0.0 0.7"/>
-    </material>
     <!-- chassis parameters -->
     <xacro:property name="bot_length" value="0.387" />
@@ -46,5 +36,5 @@
             </geometry>
             <origin xyz="0.0 0.0 ${z_offset+bot_height/2}"/>
-            <material name="white"/>
+            <material name="orange"/>
         </visual>
         <collision>
@@ -61,5 +51,5 @@
                 <box size="${bot_length} ${bot_width} ${bot_height}"/>
             </geometry>
-            <material name="white"/>
+            <material name="orange"/>
         </visual>
         <collision>
@@ -75,5 +65,5 @@
                 <box size="${bot_length} ${bot_width} ${bot_height}"/>
             </geometry>
-            <material name="white"/>
+            <material name="orange"/>
         </visual>
         <collision>
@@ -134,5 +124,5 @@
                     <box size="${pillar_length} ${pillar_width} ${pillar_height_1}"/>
                 </geometry>
-                <material name="black"/>
+                <material name="white"/>
             </visual>
             <collision>
@@ -148,5 +138,5 @@
                     <box size="${pillar_length} ${pillar_width} ${pillar_height_2}"/>
                 </geometry>
-                <material name="black"/>
+                <material name="white"/>
             </visual>
             <collision>
@@ -173,5 +163,5 @@
                     <cylinder radius="${motor_radius}" length="${motor_length}"/>
                 </geometry>
-                <material name="red"/>
+                <material name="black"/>
                 <origin rpy="${PI/2} 0.0 0.0"/>
             </visual>

File: src/bot_description/urdf/bot_gazebo.xacro (robot description, xacro)
@@ -174,3 +174,16 @@
         <material>Gazebo/Black</material>
     </gazebo>
+    <!-- lidar -->
+    <gazebo reference="lidarbase">
+        <material>Gazebo/Black</material>
+    </gazebo>
+    <gazebo reference="lidar">
+        <selfCollide>false</selfCollide>
+        <gravity>true</gravity>
+        <mu1>30</mu1>
+        <mu2>30</mu2>
+        <kp>1e60</kp>
+        <kd>1e50</kd>
+        <material>Gazebo/Purple</material>
+    </gazebo>
 </robot>

File: src/bot_description/urdf/bot_gazebo_plugin.xacro (robot description, xacro)
@@ -4,22 +4,22 @@
 	<gazebo>
 		<plugin name="bot_diff_drive" filename="libgazebo_mecanum_drive.so">
-		<commandTopic>cmd_vel</commandTopic>
-		<odometryTopic>odom</odometryTopic>
-		<odometryFrame>odom</odometryFrame>
-		<robotBaseFrame>base_link_1</robotBaseFrame>
-		<LeftRear>back_left_joint</LeftRear>
-		<LeftFront>front_left_joint</LeftFront>
-		<RightFront>front_right_joint</RightFront>
-		<RightRear>back_right_joint</RightRear>
-		<odometryRate>30</odometryRate>
-		<publishWheelTF>false</publishWheelTF>
-		<publishOdomTF>false</publishOdomTF>
-		<WheelTorque>30</WheelTorque>
-		<WheelSeparationW>0.35</WheelSeparationW>
-		<WheelSeparationL>0.6</WheelSeparationL>
-		<wheelAccel>10</wheelAccel>
-		<wheelDiameter>0.13</wheelDiameter>
-		<publishOdom>true</publishOdom>
-		<isRollerModel>true</isRollerModel>
+			<commandTopic>cmd_vel</commandTopic>
+			<odometryTopic>odom</odometryTopic>
+			<odometryFrame>odom</odometryFrame>
+			<robotBaseFrame>base_link_1</robotBaseFrame>
+			<LeftRear>back_left_joint</LeftRear>
+			<LeftFront>front_left_joint</LeftFront>
+			<RightFront>front_right_joint</RightFront>
+			<RightRear>back_right_joint</RightRear>
+			<odometryRate>30</odometryRate>
+			<publishWheelTF>false</publishWheelTF>
+			<publishOdomTF>false</publishOdomTF>
+			<WheelTorque>30</WheelTorque>
+			<WheelSeparationW>0.35</WheelSeparationW>
+			<WheelSeparationL>0.6</WheelSeparationL>
+			<wheelAccel>10</wheelAccel>
+			<wheelDiameter>0.13</wheelDiameter>
+			<publishOdom>true</publishOdom>
+			<isRollerModel>true</isRollerModel>
 		</plugin>
 	</gazebo>
@@ -27,66 +27,103 @@
 	<gazebo>
 		<plugin name="bot_joint_state" filename="libgazebo_ros_joint_state_publisher.so">
-		<ros>
-			<remapping>joint_states:=joint_states</remapping>
-		</ros>
-		<update_rate>30</update_rate>
-		<!-- wheel joint -->
-		<joint_name>back_left_joint</joint_name>
-		<joint_name>front_left_joint</joint_name>
-		<joint_name>front_right_joint</joint_name>
-		<joint_name>back_right_joint</joint_name>
-		<!-- roller front_left -->
-		<joint_name>front_left_roller_2_joint</joint_name>
-		<joint_name>front_left_roller_1_joint</joint_name>
-		<joint_name>front_left_roller_3_joint</joint_name>
-		<joint_name>front_left_roller_4_joint</joint_name>
-		<joint_name>front_left_roller_5_joint</joint_name>
-		<joint_name>front_left_roller_6_joint</joint_name>
-		<joint_name>front_left_roller_7_joint</joint_name>
-		<joint_name>front_left_roller_8_joint</joint_name>
-		<joint_name>front_left_roller_9_joint</joint_name>
-		<joint_name>front_left_roller_10_joint</joint_name>
-		<joint_name>front_left_roller_11_joint</joint_name>
-		<joint_name>front_left_roller_12_joint</joint_name>
-		<!-- roller back_left -->
-		<joint_name>back_left_roller_2_joint</joint_name>
-		<joint_name>back_left_roller_1_joint</joint_name>
-		<joint_name>back_left_roller_3_joint</joint_name>
-		<joint_name>back_left_roller_4_joint</joint_name>
-		<joint_name>back_left_roller_5_joint</joint_name>
-		<joint_name>back_left_roller_6_joint</joint_name>
-		<joint_name>back_left_roller_7_joint</joint_name>
-		<joint_name>back_left_roller_8_joint</joint_name>
-		<joint_name>back_left_roller_9_joint</joint_name>
-		<joint_name>back_left_roller_10_joint</joint_name>
-		<joint_name>back_left_roller_11_joint</joint_name>
-		<joint_name>back_left_roller_12_joint</joint_name>
-		<!-- roller back_right -->
-		<joint_name>back_right_roller_2_joint</joint_name>
-		<joint_name>back_right_roller_1_joint</joint_name>
-		<joint_name>back_right_roller_3_joint</joint_name>
-		<joint_name>back_right_roller_4_joint</joint_name>
-		<joint_name>back_right_roller_5_joint</joint_name>
-		<joint_name>back_right_roller_6_joint</joint_name>
-		<joint_name>back_right_roller_7_joint</joint_name>
-		<joint_name>back_right_roller_8_joint</joint_name>
-		<joint_name>back_right_roller_9_joint</joint_name>
-		<joint_name>back_right_roller_10_joint</joint_name>
-		<joint_name>back_right_roller_11_joint</joint_name>
-		<joint_name>back_right_roller_12_joint</joint_name>
-		<!-- roller front_right -->
-		<joint_name>front_right_roller_2_joint</joint_name>
-		<joint_name>front_right_roller_1_joint</joint_name>
-		<joint_name>front_right_roller_3_joint</joint_name>
-		<joint_name>front_right_roller_4_joint</joint_name>
-		<joint_name>front_right_roller_5_joint</joint_name>
-		<joint_name>front_right_roller_6_joint</joint_name>
-		<joint_name>front_right_roller_7_joint</joint_name>
-		<joint_name>front_right_roller_8_joint</joint_name>
-		<joint_name>front_right_roller_9_joint</joint_name>
-		<joint_name>front_right_roller_10_joint</joint_name>
-		<joint_name>front_right_roller_11_joint</joint_name>
-		<joint_name>front_right_roller_12_joint</joint_name>
+			<ros>
+				<remapping>joint_states:=joint_states</remapping>
+			</ros>
+			<update_rate>30</update_rate>
+			<!-- wheel joint -->
+			<joint_name>back_left_joint</joint_name>
+			<joint_name>front_left_joint</joint_name>
+			<joint_name>front_right_joint</joint_name>
+			<joint_name>back_right_joint</joint_name>
+			<!-- roller front_left -->
+			<joint_name>front_left_roller_2_joint</joint_name>
+			<joint_name>front_left_roller_1_joint</joint_name>
+			<joint_name>front_left_roller_3_joint</joint_name>
+			<joint_name>front_left_roller_4_joint</joint_name>
+			<joint_name>front_left_roller_5_joint</joint_name>
+			<joint_name>front_left_roller_6_joint</joint_name>
+			<joint_name>front_left_roller_7_joint</joint_name>
+			<joint_name>front_left_roller_8_joint</joint_name>
+			<joint_name>front_left_roller_9_joint</joint_name>
+			<joint_name>front_left_roller_10_joint</joint_name>
+			<joint_name>front_left_roller_11_joint</joint_name>
+			<joint_name>front_left_roller_12_joint</joint_name>
+			<!-- roller back_left -->
+			<joint_name>back_left_roller_2_joint</joint_name>
+			<joint_name>back_left_roller_1_joint</joint_name>
+			<joint_name>back_left_roller_3_joint</joint_name>
+			<joint_name>back_left_roller_4_joint</joint_name>
+			<joint_name>back_left_roller_5_joint</joint_name>
+			<joint_name>back_left_roller_6_joint</joint_name>
+			<joint_name>back_left_roller_7_joint</joint_name>
+			<joint_name>back_left_roller_8_joint</joint_name>
+			<joint_name>back_left_roller_9_joint</joint_name>
+			<joint_name>back_left_roller_10_joint</joint_name>
+			<joint_name>back_left_roller_11_joint</joint_name>
+			<joint_name>back_left_roller_12_joint</joint_name>
+			<!-- roller back_right -->
+			<joint_name>back_right_roller_2_joint</joint_name>
+			<joint_name>back_right_roller_1_joint</joint_name>
+			<joint_name>back_right_roller_3_joint</joint_name>
+			<joint_name>back_right_roller_4_joint</joint_name>
+			<joint_name>back_right_roller_5_joint</joint_name>
+			<joint_name>back_right_roller_6_joint</joint_name>
+			<joint_name>back_right_roller_7_joint</joint_name>
+			<joint_name>back_right_roller_8_joint</joint_name>
+			<joint_name>back_right_roller_9_joint</joint_name>
+			<joint_name>back_right_roller_10_joint</joint_name>
+			<joint_name>back_right_roller_11_joint</joint_name>
+			<joint_name>back_right_roller_12_joint</joint_name>
+			<!-- roller front_right -->
+			<joint_name>front_right_roller_2_joint</joint_name>
+			<joint_name>front_right_roller_1_joint</joint_name>
+			<joint_name>front_right_roller_3_joint</joint_name>
+			<joint_name>front_right_roller_4_joint</joint_name>
+			<joint_name>front_right_roller_5_joint</joint_name>
+			<joint_name>front_right_roller_6_joint</joint_name>
+			<joint_name>front_right_roller_7_joint</joint_name>
+			<joint_name>front_right_roller_8_joint</joint_name>
+			<joint_name>front_right_roller_9_joint</joint_name>
+			<joint_name>front_right_roller_10_joint</joint_name>
+			<joint_name>front_right_roller_11_joint</joint_name>
+			<joint_name>front_right_roller_12_joint</joint_name>
 		</plugin>
 	</gazebo>
+	<!-- sick LiDAR 0 controller -->
+	<gazebo reference="lidar">
+		<sensor type="ray" name="sllidar_sensor">
+			<pose>0 0 0 0 0 0</pose>
+			<always_on>false</always_on>
+			<visualize>false</visualize>
+			<update_rate>40</update_rate>
+			<ray>
+				<scan>
+					<horizontal>
+						<samples>720</samples>
+						<resolution>1</resolution>
+						<min_angle>-2.35619445</min_angle>
+						<max_angle>2.35619445</max_angle>
+					</horizontal>
+				</scan>
+				<range>
+					<min>0.10</min>
+					<max>30.0</max>
+					<resolution>0.01</resolution>
+				</range>
+				<noise>
+					<type>gaussian</type>
+					<mean>0.0</mean>
+					<stddev>0.01</stddev>
+				</noise>
+			</ray>
+			<plugin name="bot_lidar_sensor" filename="libgazebo_ros_ray_sensor.so">
+				<ros>
+					<!-- <namespace>/tb3</namespace> -->
+					<remapping>~/out:=/scan</remapping>
+				</ros>
+				<output_type>sensor_msgs/LaserScan</output_type>
+				<frame_name>lidar</frame_name>
+			</plugin>
+		</sensor>
+	</gazebo>
 </robot>

File: src/bot_description/urdf/bot_wheel.urdf.xacro (robot description, xacro)
@@ -22,7 +22,5 @@
             <cylinder radius="${wheel_radius}" length="${wheel_width}"/>
             </geometry>
-            <material name="white">
-                        <color rgba="1 1 0.9 1"/>
-            </material>
+            <material name="white"/>
         </visual>
         <collision>
@@ -43,7 +41,5 @@
                     <cylinder radius="${roller_radius}" length="${roller_length}"/>
                     </geometry>
-                    <material name="black">
-                        <color rgba="0.1 0.1 0.1 1"/>
-                    </material>
+                    <material name="black"/>
                 </visual>
                 <collision>
