Commit message: add base_footprint

File: src/bot_description/urdf/bot.urdf.xacro (robot description, xacro)
@@ -7,5 +7,3 @@
     <xacro:include filename="bot_gazebo.xacro"/>
     <xacro:include filename="bot_gazebo_plugin.xacro"/>
-    <!-- <xacro:include filename="$(find bot_description)/ros2_control/bot_control.xacro"/>
-    <xacro:bot_ros2_control/> -->
 </robot>

File: src/bot_description/urdf/bot_base.urdf.xacro (robot description, xacro)
@@ -24,9 +24,10 @@
     <xacro:property name="wheel_joint_x" value="${bot_length/2 - 0.045}" />
     <xacro:property name="wheel_joint_y" value="${bot_width/2 + wheel_base_dis + wheel_length/2}" />
-    <xacro:property name="wheel_joint_z" value="${wheel_radius}" />
+    <xacro:property name="wheel_joint_z" value="${wheel_radius-z_offset}" />
     <!-- motor parameters -->
-    <xacro:property name="motor_radius" value="${wheel_radius-z_offset-bot_height}" />
+    <xacro:property name="motor_radius" value="${wheel_radius-z_offset}" />
     <xacro:property name="motor_length" value="0.12" />
     <xacro:property name="motor_mass" value="0.3" />
+    <link name="base_footprint"/>
     <!--   Define three chassis base_link_1 base_link_2 base_link_3-->
     <link name="base_link_1">
@@ -35,5 +36,4 @@
                 <box size="${bot_length} ${bot_width} ${bot_height}"/>
             </geometry>
-            <origin xyz="0.0 0.0 ${z_offset+bot_height/2}"/>
             <material name="orange"/>
         </visual>
@@ -42,8 +42,12 @@
                 <box size="${bot_length} ${bot_width} ${bot_height}"/>
             </geometry>
-            <origin xyz="0.0 0.0 ${z_offset}"/>
         </collision>
         <xacro:box_inertial_matrix mass="${bot_mass}" length="${bot_length}" width="${bot_width}" height="${bot_height}" />
     </link>
+    <joint name="base_joint" type="fixed">
+        <parent link="base_footprint"/>
+        <child link="base_link_1"/>
+        <origin xyz="0.0 0.0 ${z_offset+bot_height/2}"/>
+    </joint>
     <link name="base_link_2">
         <visual>
@@ -77,5 +81,5 @@
         <parent link="base_link_1"/>
         <child link="base_link_2"/>
-        <origin xyz="0.0 0.0 ${pillar_height_1+z_offset+bot_height/2*3}"/>
+        <origin xyz="0.0 0.0 ${pillar_height_1+bot_height}"/>
     </joint>
     <joint name="base23_joint" type="fixed">
@@ -150,5 +154,5 @@
             <parent link="base_link_1"/>
             <child link="${link_name}_p1"/>
-            <origin xyz="${(bot_length/2-pillar_length/2) * front_flag} ${(bot_width/3) * left_flag} ${z_offset+bot_height+pillar_height_1/2}"/>
+            <origin xyz="${(bot_length/2-pillar_length/2) * front_flag} ${(bot_width/3) * left_flag} ${bot_height/2+pillar_height_1/2}"/>
         </joint>
         <joint name="${link_name}_p2base_joint" type="fixed">

File: src/bot_description/urdf/bot_gazebo_plugin.xacro (robot description, xacro)
@@ -7,5 +7,5 @@
 			<odometryTopic>odom</odometryTopic>
 			<odometryFrame>odom</odometryFrame>
-			<robotBaseFrame>base_link_1</robotBaseFrame>
+			<robotBaseFrame>base_footprint</robotBaseFrame>
 			<LeftRear>back_left_joint</LeftRear>
 			<LeftFront>front_left_joint</LeftFront>

File: src/bot_description/urdf/bot_wheel.urdf.xacro (robot description, xacro)
@@ -2,11 +2,12 @@
 <robot xmlns:xacro="http://ros.org/wiki/xacro">
     <!-- Properties -->
-    <xacro:property name="wheel_radius" value="0.0635" />
-    <xacro:property name="wheel_width" value="0.05" />
-    <xacro:property name="wheel_mass" value="0.5" />
     <xacro:property name="roller_mass" value="0.02"/>
     <xacro:property name="roller_radius" value="0.008"/>
     <xacro:property name="roller_length" value="0.046"/>
     <xacro:property name="roller_number" value="12"/>
+    <xacro:property name="wheel_radius" value="0.0635" />
+    <xacro:property name="wheel_internal_radius" value="${wheel_radius-roller_radius/2}" />
+    <xacro:property name="wheel_width" value="0.05" />
+    <xacro:property name="wheel_mass" value="0.5" />
     <!-- Mecanum Wheel Macro -->
     <xacro:macro name="mecanum_wheel" params="name roller_angle">
@@ -20,5 +21,5 @@
         <visual>
             <geometry>
-            <cylinder radius="${wheel_radius}" length="${wheel_width}"/>
+            <cylinder radius="${wheel_internal_radius}" length="${wheel_width}"/>
             </geometry>
             <material name="white"/>
@@ -26,5 +27,5 @@
         <collision>
             <geometry>
-            <cylinder radius="${wheel_radius}" length="${wheel_width}"/>
+            <cylinder radius="${wheel_internal_radius}" length="${wheel_width}"/>
             </geometry>
         </collision>
@@ -57,5 +58,5 @@
                 <child link="${name}"/>
                 <origin
-                    xyz="${wheel_radius*cos(angle)} ${wheel_radius*sin(angle)} 0"
+                    xyz="${wheel_internal_radius*cos(angle)} ${wheel_internal_radius*sin(angle)} 0"
                     rpy="${roller_angle} 0 ${angle}"/>
                 <axis xyz="0 0 1"/>

File: src/bot_description/urdf/material.urdf.xacro (robot description, xacro)
@@ -1,5 +1,5 @@
 <?xml version="1.0"?>
 <robot xmlns:xacro="http://www.ros.org/wiki/xacro">
-    <xacro:property name="alpha" value="0.8" />
+    <xacro:property name="alpha" value="1.0" />
     <material name="red">           <color rgba="${255/255}  ${0/255  } ${0/255  }  ${alpha}"/>    </material>
     <material name="redbright">     <color rgba="${255/255}  ${51/255 } ${51/255 }  ${alpha}"/>    </material>

Commit message: feat:add camera

File: src/bot_description/urdf/bot.urdf.xacro (robot description, xacro)
@@ -5,4 +5,5 @@
     <xacro:include filename="bot_base.urdf.xacro"/>
     <xacro:include filename="bot_lidar.urdf.xacro"/>
+    <xacro:include filename="bot_camera.urdf.xacro"/>
     <xacro:include filename="bot_gazebo.xacro"/>
     <xacro:include filename="bot_gazebo_plugin.xacro"/>

File: src/bot_description/urdf/bot_gazebo.xacro (robot description, xacro)
@@ -187,3 +187,28 @@
         <material>Gazebo/Purple</material>
     </gazebo>
+    <!-- camera -->
+    <gazebo reference="foothold_base_1">
+        <material>Gazebo/Black</material>
+    </gazebo>
+    <gazebo reference="foothold_base_2">
+        <material>Gazebo/Black</material>
+    </gazebo>
+    <gazebo reference="foothold_base_3">
+        <material>Gazebo/Black</material>
+    </gazebo>
+    <gazebo reference="foothold_base_4">
+        <material>Gazebo/Black</material>
+    </gazebo>
+    <gazebo reference="camera_link">
+        <material>Gazebo/Black</material>
+    </gazebo>
+    <gazebo reference="camera">
+        <selfCollide>false</selfCollide>
+        <gravity>true</gravity>
+        <mu1>30</mu1>
+        <mu2>30</mu2>
+        <kp>1e60</kp>
+        <kd>1e50</kd>
+        <material>Gazebo/White</material>
+    </gazebo>
 </robot>

File: src/bot_description/urdf/bot_gazebo_plugin.xacro (robot description, xacro)
@@ -1,5 +1,5 @@
 <?xml version="1.0"?>
 <robot xmlns:xacro="http://www.ros.org/wiki/xacro">
-	<!-- gazebo_mecanum plugin -->
+	<!-- import gazebo_mecanum_drive plugin -->
 	<gazebo>
 		<plugin name="bot_diff_drive" filename="libgazebo_mecanum_drive.so">
@@ -24,5 +24,5 @@
 		</plugin>
 	</gazebo>
-	<!-- gazebo joint_state_publisher -->
+	<!-- import joint_state_publisher plugin -->
 	<gazebo>
 		<plugin name="bot_joint_state" filename="libgazebo_ros_joint_state_publisher.so">
@@ -90,5 +90,5 @@
 		</plugin>
 	</gazebo>
-	<!-- sick LiDAR 0 controller -->
+	<!-- import lidar controller plugin -->
 	<gazebo reference="lidar">
 		<sensor type="ray" name="sllidar_sensor">
@@ -127,3 +127,29 @@
 		</sensor>
 	</gazebo>
+	<!-- import camera controller plugin -->
+	<gazebo reference="camera">
+		<sensor name="camera" type="camera">
+		<always_on>true</always_on>
+		<visualize>true</visualize>
+		<update_rate>30</update_rate>
+		<camera name="camera">
+			<horizontal_fov>1.047198</horizontal_fov>
+			<image>
+			<width>960</width>
+			<height>540</height>
+			<format>R8G8B8</format>
+			</image>
+			<clip>
+			<near>0.1</near>
+			<far>10</far>
+			</clip>
+		</camera>
+		<plugin name="camera_driver" filename="libgazebo_ros_camera.so">
+			<camera_name>camera</camera_name>
+			<frame_name>camera</frame_name>
+			<triggered>false</triggered>
+			<hack_baseline>0.07</hack_baseline>
+		</plugin>
+		</sensor>
+	</gazebo>
 </robot>

Commit message: feat:add realsense depth camera

File: src/bot_description/urdf/bot.urdf.xacro (robot description, xacro)
@@ -6,4 +6,8 @@
     <xacro:include filename="bot_lidar.urdf.xacro"/>
     <xacro:include filename="bot_camera.urdf.xacro"/>
+    <xacro:include filename="bot_depth.urdf.xacro"/>
+    <xacro:sensor_d455 parent="base_link_3" use_nominal_extrinsics="false">
+        <origin xyz="${bot_length/2-0.026/2} 0 ${bot_height/2}" rpy="0 0 0"/>
+    </xacro:sensor_d455>
     <xacro:include filename="bot_gazebo.xacro"/>
     <xacro:include filename="bot_gazebo_plugin.xacro"/>

File: src/bot_description/urdf/bot_gazebo.xacro (robot description, xacro)
@@ -212,3 +212,13 @@
         <material>Gazebo/White</material>
     </gazebo>
+    <!-- depth camera -->
+    <gazebo reference="depth_link">
+        <selfCollide>false</selfCollide>
+        <gravity>true</gravity>
+        <mu1>30</mu1>
+        <mu2>30</mu2>
+        <kp>1e60</kp>
+        <kd>1e50</kd>
+        <material>Gazebo/Grey</material>
+    </gazebo>
 </robot>

File: src/bot_description/urdf/bot_gazebo_plugin.xacro (robot description, xacro)
@@ -127,11 +127,11 @@
 		</sensor>
 	</gazebo>
-	<!-- import camera controller plugin -->
-	<gazebo reference="camera">
-		<sensor name="camera" type="camera">
+	<!-- import depth camera controller plugin -->
+	<gazebo reference="depth_link">
+		<sensor name="depth_camera" type="depth">
 		<always_on>true</always_on>
 		<visualize>true</visualize>
 		<update_rate>30</update_rate>
-		<camera name="camera">
+		<camera name="depth_camera">
 			<horizontal_fov>1.047198</horizontal_fov>
 			<image>
@@ -141,9 +141,9 @@
 			</image>
 			<clip>
-			<near>0.1</near>
-			<far>10</far>
+			<near>0.05</near>
+			<far>3</far>
 			</clip>
 		</camera>
-		<plugin name="camera_driver" filename="libgazebo_ros_camera.so">
+		<plugin name="depth_camera_driver" filename="libgazebo_ros_camera.so">
 			<camera_name>camera</camera_name>
 			<frame_name>camera</frame_name>

File: src/bot_description/urdf/material.urdf.xacro (robot description, xacro)
@@ -19,4 +19,5 @@
     <material name="grey">          <color rgba="${128/255}  ${128/255} ${128/255}  ${alpha}"/>    </material>
     <material name="darkgrey">      <color rgba="${64/255 }  ${64/255 } ${64/255 }  ${alpha}"/>    </material>
+    <material name="plastic">       <color rgba="0.1 0.1 0.1 1"/>                                  </material>
 </robot>
 <!--
@@ -38,3 +39,4 @@
     灰色 (Grey): RGB(128, 128, 128)
     深灰色 (DarkGrey): RGB(64, 64, 64)
+    塑料(plastic)
  -->

Commit message: feat:imu_n100

File: src/bot_description/urdf/bot.urdf.xacro (robot description, xacro)
@@ -10,4 +10,8 @@
         <origin xyz="${bot_length/2-0.026/2} 0 ${bot_height/2}" rpy="0 0 0"/>
     </xacro:sensor_d455>
+    <xacro:include filename="bot_imu.urdf.xacro"/>
+    <xacro:imu_n100 parent="base_link_2">
+        <origin xyz="0 0 ${bot_height/2}" rpy="0 0 0"/>
+    </xacro:imu_n100>
     <xacro:include filename="bot_gazebo.xacro"/>
     <xacro:include filename="bot_gazebo_plugin.xacro"/>

File: src/bot_description/urdf/bot_gazebo.xacro (robot description, xacro)
@@ -222,3 +222,9 @@
         <material>Gazebo/Grey</material>
     </gazebo>
+    <gazebo reference="n100_base_link">
+        <material>Gazebo/Grey</material>
+    </gazebo>
+    <gazebo reference="imu_n100">
+        <material>Gazebo/Grey</material>
+    </gazebo>
 </robot>

File: src/bot_description/urdf/bot_gazebo_plugin.xacro (robot description, xacro)
@@ -102,6 +102,7 @@
 						<samples>720</samples>
 						<resolution>1</resolution>
-						<min_angle>-2.35619445</min_angle>
-						<max_angle>2.35619445</max_angle>
+						<!-- 45/180*pi -->
+						<min_angle>-0.785398</min_angle>
+						<max_angle>0.785398</max_angle>
 					</horizontal>
 				</scan>
@@ -153,3 +154,56 @@
 		</sensor>
 	</gazebo>
+	<gazebo reference="imu_n100">
+		<sensor name="imu_sensor" type="imu">
+		<always_on>true</always_on>
+		<update_rate>30</update_rate>
+		<imu>
+			<angular_velocity>
+			<x>
+				<noise type="gaussian">
+				<mean>0.0</mean>
+				<stddev>2e-4</stddev>
+				</noise>
+			</x>
+			<y>
+				<noise type="gaussian">
+				<mean>0.0</mean>
+				<stddev>2e-4</stddev>
+				</noise>
+			</y>
+			<z>
+				<noise type="gaussian">
+				<mean>0.0</mean>
+				<stddev>2e-4</stddev>
+				</noise>
+			</z>
+			</angular_velocity>
+			<linear_acceleration>
+			<x>
+				<noise type="gaussian">
+				<mean>0.0</mean>
+				<stddev>1.7e-2</stddev>
+				</noise>
+			</x>
+			<y>
+				<noise type="gaussian">
+				<mean>0.0</mean>
+				<stddev>1.7e-2</stddev>
+				</noise>
+			</y>
+				<z>
+				<noise type="gaussian">
+				<mean>0.0</mean>
+				<stddev>1.7e-2</stddev>
+				</noise>
+			</z>
+			</linear_acceleration>
+		</imu>
+		<plugin filename="libgazebo_ros_imu_sensor.so" name="imu_plugin">
+			<ros>
+			<remapping>~/out:=imu_n100</remapping>
+			</ros>
+		</plugin>
+		</sensor>
+	</gazebo>
 </robot>
