Commit message: feat:use cartographer to build map

File: src/bot_description/urdf/bot.urdf.xacro (robot description, xacro)
@@ -4,14 +4,22 @@
     <xacro:include filename="bot_wheel.urdf.xacro"/>
     <xacro:include filename="bot_base.urdf.xacro"/>
+    <!-- add camera -->
+    <xacro:include filename="bot_camera.urdf.xacro"/>
+    <!-- add lidar -->
     <xacro:include filename="bot_lidar.urdf.xacro"/>
-    <xacro:include filename="bot_camera.urdf.xacro"/>
+    <xacro:lidar_func parent="base_link_3">
+        <origin xyz="${bot_length/2-lidar_radius} 0 ${bot_height/2+lidar_height/4}" rpy="0 0 0"/>
+    </xacro:lidar_func>
+    <!-- add depth camera -->
     <xacro:include filename="bot_depth.urdf.xacro"/>
-    <xacro:sensor_d455 parent="base_link_3" use_nominal_extrinsics="false">
-        <origin xyz="${bot_length/2-0.026/2} 0 ${bot_height/2}" rpy="0 0 0"/>
+    <xacro:sensor_d455 parent="base_link_2" use_nominal_extrinsics="false">
+        <origin xyz="${bot_length/2-d455_cam_depth/2} 0 ${bot_height/2}" rpy="0 0 0"/>
     </xacro:sensor_d455>
+    <!-- add imu -->
     <xacro:include filename="bot_imu.urdf.xacro"/>
     <xacro:imu_n100 parent="base_link_2">
         <origin xyz="0 0 ${bot_height/2}" rpy="0 0 0"/>
     </xacro:imu_n100>
+    <!-- load gazebo plugins -->
     <xacro:include filename="bot_gazebo.xacro"/>
     <xacro:include filename="bot_gazebo_plugin.xacro"/>

File: src/bot_description/urdf/bot_depth.urdf.xacro (robot description, xacro)
@@ -20,29 +20,29 @@
 -->
 <robot name="sensor_d455" xmlns:xacro="http://ros.org/wiki/xacro">
+  <!-- The following values are approximate, and the camera node
+    publishing TF values with actual calibrated camera extrinsic values -->
+  <xacro:property name="d455_cam_depth_to_infra1_offset" value="0.0"/>
+  <xacro:property name="d455_cam_depth_to_infra2_offset" value="-0.095"/>
+  <xacro:property name="d455_cam_depth_to_color_offset" value="-0.059"/>
+  <!-- The following values model the grey peripherial case for the
+  d455 camera, with the camera joint represented by the actual
+  peripherial camera tripod mount -->
+  <xacro:property name="d455_cam_width" value="0.124"/>
+  <xacro:property name="d455_cam_height" value="0.029"/>
+  <xacro:property name="d455_cam_depth" value="0.026"/>
+  <xacro:property name="d455_cam_mount_from_center_offset" value="0.0158"/>
+  <!-- glass cover is 0.1 mm inwards from front aluminium plate -->
+  <xacro:property name="d455_glass_to_front" value="0.1e-3"/>
+  <!-- see datasheet Revision 009, Fig. 4-4 page 68 -->
+  <xacro:property name="d455_zero_depth_to_glass" value="4.55e-3"/>
+  <!-- convenience precomputation to avoid clutter-->
+  <xacro:property name="d455_mesh_x_offset" value="${d455_cam_mount_from_center_offset-d455_glass_to_front-d455_zero_depth_to_glass}"/>
+  <!-- The following offset is relative to the physical d455 camera peripherial
+  camera tripod mount -->
+  <xacro:property name="d455_cam_depth_px" value="${d455_cam_mount_from_center_offset}"/>
+  <xacro:property name="d455_cam_depth_py" value="0.0475"/>
+  <xacro:property name="d455_cam_depth_pz" value="${d455_cam_height/2}"/>
   <xacro:macro name="sensor_d455" params="parent *origin name:=depth use_nominal_extrinsics:=false">
     <xacro:property name="M_PI" value="3.1415926535897931" />
-    <!-- The following values are approximate, and the camera node
-     publishing TF values with actual calibrated camera extrinsic values -->
-    <xacro:property name="d455_cam_depth_to_infra1_offset" value="0.0"/>
-    <xacro:property name="d455_cam_depth_to_infra2_offset" value="-0.095"/>
-    <xacro:property name="d455_cam_depth_to_color_offset" value="-0.059"/>
-    <!-- The following values model the grey peripherial case for the
-  	d455 camera, with the camera joint represented by the actual
-  	peripherial camera tripod mount -->
-    <xacro:property name="d455_cam_width" value="0.124"/>
-    <xacro:property name="d455_cam_height" value="0.029"/>
-    <xacro:property name="d455_cam_depth" value="0.026"/>
-    <xacro:property name="d455_cam_mount_from_center_offset" value="0.0158"/>
-    <!-- glass cover is 0.1 mm inwards from front aluminium plate -->
-    <xacro:property name="d455_glass_to_front" value="0.1e-3"/>
-    <!-- see datasheet Revision 009, Fig. 4-4 page 68 -->
-    <xacro:property name="d455_zero_depth_to_glass" value="4.55e-3"/>
-    <!-- convenience precomputation to avoid clutter-->
-    <xacro:property name="d455_mesh_x_offset" value="${d455_cam_mount_from_center_offset-d455_glass_to_front-d455_zero_depth_to_glass}"/>
-    <!-- The following offset is relative to the physical d455 camera peripherial
-  	camera tripod mount -->
-    <xacro:property name="d455_cam_depth_px" value="${d455_cam_mount_from_center_offset}"/>
-    <xacro:property name="d455_cam_depth_py" value="0.0475"/>
-    <xacro:property name="d455_cam_depth_pz" value="${d455_cam_height/2}"/>
     <!-- camera body, with origin at bottom screw mount -->
     <joint name="${name}_joint" type="fixed">

File: src/bot_description/urdf/bot_gazebo_plugin.xacro (robot description, xacro)
@@ -28,5 +28,5 @@
 		<plugin name="bot_joint_state" filename="libgazebo_ros_joint_state_publisher.so">
 			<ros>
-				<remapping>joint_states:=joint_states</remapping>
+				<remapping>~/out:=joint_states</remapping>
 			</ros>
 			<update_rate>30</update_rate>
@@ -94,21 +94,21 @@
 		<sensor type="ray" name="sllidar_sensor">
 			<pose>0 0 0 0 0 0</pose>
-			<always_on>false</always_on>
-			<visualize>false</visualize>
-			<update_rate>40</update_rate>
+			<always_on>true</always_on>
+			<visualize>true</visualize>
+			<update_rate>30</update_rate>
 			<ray>
 				<scan>
 					<horizontal>
-						<samples>720</samples>
+						<samples>360</samples>
 						<resolution>1</resolution>
-						<!-- 45/180*pi -->
-						<min_angle>-0.785398</min_angle>
-						<max_angle>0.785398</max_angle>
+						<!-- 135/180*pi -->
+						<min_angle>-2.356194</min_angle>
+						<max_angle>2.356194</max_angle>
 					</horizontal>
 				</scan>
 				<range>
-					<min>0.10</min>
-					<max>30.0</max>
-					<resolution>0.01</resolution>
+					<min>0.12000</min>
+					<max>11</max>
+					<resolution>0.015000</resolution>
 				</range>
 				<noise>
@@ -120,5 +120,4 @@
 			<plugin name="bot_lidar_sensor" filename="libgazebo_ros_ray_sensor.so">
 				<ros>
-					<!-- <namespace>/tb3</namespace> -->
 					<remapping>~/out:=/scan</remapping>
 				</ros>
@@ -154,8 +153,9 @@
 		</sensor>
 	</gazebo>
+	<!-- import imu controller plugin -->
 	<gazebo reference="imu_n100">
 		<sensor name="imu_sensor" type="imu">
 		<always_on>true</always_on>
-		<update_rate>30</update_rate>
+		<update_rate>200</update_rate>
 		<imu>
 			<angular_velocity>
@@ -202,5 +202,5 @@
 		<plugin filename="libgazebo_ros_imu_sensor.so" name="imu_plugin">
 			<ros>
-			<remapping>~/out:=imu_n100</remapping>
+			<remapping>~/out:=imu</remapping>
 			</ros>
 		</plugin>

File: src/bot_description/urdf/bot_lidar.urdf.xacro (robot description, xacro)
@@ -1,48 +1,53 @@
-<robot xmlns:xacro="http://www.ros.org/wiki/xacro">
+<robot name="lidar" xmlns:xacro="http://www.ros.org/wiki/xacro">
     <xacro:property name="lidar_radius" value="0.038" />
     <xacro:property name="lidar_height" value="0.04" />
-    <xacro:property name="lidar_joint_x" value="${bot_length/2-0.055}" />
-    <xacro:property name="lidar_joint_y" value="0" />
-    <xacro:property name="lidar_joint_z" value="${bot_height/2+lidar_height/4}" />
-    <link name="lidarbase">
-        <visual>
-            <geometry>
-                <cylinder radius="${lidar_radius}" length="${lidar_height/2}"/>
-            </geometry>
-            <material name="black">
-                <color rgba="0.1 0.1 0.1 0.8"/>
-            </material>
-        </visual>
-        <collision>
-            <geometry>
-                <cylinder radius="${lidar_radius}" length="${lidar_height/2}"/>
-            </geometry>
-        </collision>
-        <xacro:cylinder_inertial_matrix mass="0.3" radius="${lidar_radius}" length="${lidar_height/2}" />
-    </link>
-    <joint name="lidarbase2base_link_2" type="fixed">
-        <parent link="base_link_2"/>
-        <child link="lidarbase"/>
-        <origin xyz="${lidar_joint_x} ${lidar_joint_y} ${lidar_joint_z}"/>
-    </joint>
-    <link name="lidar">
-        <visual>
-            <geometry>
-                <cylinder radius="${lidar_radius}" length="${lidar_height/2}"/>
-            </geometry>
-            <material name="purple"/>
-        </visual>
-        <collision>
-            <geometry>
-                <cylinder radius="${lidar_radius}" length="${lidar_height/2}"/>
-            </geometry>
-        </collision>
-        <xacro:cylinder_inertial_matrix mass="0.3" radius="${lidar_radius}" length="${lidar_height/2}" />
-    </link>
-    <joint name="lidar_joint" type="fixed">
-        <parent link="lidarbase"/>
-        <child link="lidar"/>
-        <origin xyz="0 0 ${lidar_height/2}"/>
-        <axis xyz="0 0 1"/>
-    </joint>
+    <xacro:macro name="lidar_func" params="parent *origin">
+        <link name="lidar_base_footprint"/>
+        <joint name="lidar_footprint_joint" type="fixed">
+            <xacro:insert_block name="origin" />
+            <parent link="${parent}"/>
+            <child link="lidar_base_footprint"/>
+        </joint>
+        <link name="lidarbase">
+            <visual>
+                <geometry>
+                    <cylinder radius="${lidar_radius}" length="${lidar_height/2}"/>
+                </geometry>
+                <material name="black">
+                    <color rgba="0.1 0.1 0.1 0.8"/>
+                </material>
+            </visual>
+            <collision>
+                <geometry>
+                    <cylinder radius="${lidar_radius}" length="${lidar_height/2}"/>
+                </geometry>
+            </collision>
+            <xacro:cylinder_inertial_matrix mass="0.3" radius="${lidar_radius}" length="${lidar_height/2}" />
+        </link>
+        <joint name="lidarbase2base_footprint" type="fixed">
+            <parent link="lidar_base_footprint"/>
+            <child link="lidarbase"/>
+            <!-- <origin xyz="${lidar_joint_x} ${lidar_joint_y} ${lidar_joint_z}"/> -->
+        </joint>
+        <link name="lidar">
+            <visual>
+                <geometry>
+                    <cylinder radius="${lidar_radius}" length="${lidar_height/2}"/>
+                </geometry>
+                <material name="purple"/>
+            </visual>
+            <collision>
+                <geometry>
+                    <cylinder radius="${lidar_radius}" length="${lidar_height/2}"/>
+                </geometry>
+            </collision>
+            <xacro:cylinder_inertial_matrix mass="0.3" radius="${lidar_radius}" length="${lidar_height/2}" />
+        </link>
+        <joint name="lidar_joint" type="fixed">
+            <parent link="lidarbase"/>
+            <child link="lidar"/>
+            <origin xyz="0 0 ${lidar_height/2}"/>
+            <axis xyz="0 0 1"/>
+        </joint>
+    </xacro:macro>
 </robot>

Commit message: modify parameters

File: src/bot_description/urdf/bot.urdf.xacro (robot description, xacro)
@@ -6,4 +6,7 @@
     <!-- add camera -->
     <xacro:include filename="bot_camera.urdf.xacro"/>
+    <xacro:camera_func parent="base_link_3">
+        <origin xyz="0 0 0" rpy="0 0 0"/>
+    </xacro:camera_func>
     <!-- add lidar -->
     <xacro:include filename="bot_lidar.urdf.xacro"/>

File: src/bot_description/urdf/bot_base.urdf.xacro (robot description, xacro)
@@ -20,11 +20,13 @@
     <xacro:property name="wheel_length" value="0.05" />
     <xacro:property name="wheel_mass" value="0.5" />
+    <xacro:property name="wheel_separation_w" value="0.36" />
+    <xacro:property name="wheel_separation_l" value="0.32" />
     <!-- wheel joint offset -->
     <xacro:property name="wheel_base_dis" value="0.03" />
-    <xacro:property name="wheel_joint_x" value="${bot_length/2 - 0.045}" />
+    <xacro:property name="wheel_joint_x" value="${wheel_separation_l/2}" />
     <xacro:property name="wheel_joint_y" value="${bot_width/2 + wheel_base_dis + wheel_length/2}" />
     <xacro:property name="wheel_joint_z" value="${wheel_radius-z_offset}" />
     <!-- motor parameters -->
-    <xacro:property name="motor_radius" value="${wheel_radius-z_offset}" />
+    <xacro:property name="motor_radius" value="${wheel_radius-z_offset-0.015}" />
     <xacro:property name="motor_length" value="0.12" />
     <xacro:property name="motor_mass" value="0.3" />

File: src/bot_description/urdf/bot_camera.urdf.xacro (robot description, xacro)
@@ -1,121 +1,129 @@
 <?xml version="1.0"?>
-<robot xmlns:xacro="http://www.ros.org/wiki/xacro">
+<robot name="camera_func" xmlns:xacro="http://www.ros.org/wiki/xacro">
     <xacro:property name="camera_radius" value="0.07" />
     <xacro:property name="foothold_radius" value="0.111" />
     <xacro:property name="foothold_height" value="0.01" />
-    <link name="foothold_base_1">
-        <visual>
-            <geometry>
-                <cylinder radius="${foothold_radius}" length="${foothold_height}"/>
-            </geometry>
-            <material name="black" />
-        </visual>
-        <collision>
-            <geometry>
-                <cylinder radius="${foothold_radius}" length="${foothold_height}"/>
-            </geometry>
-        </collision>
-        <xacro:cylinder_inertial_matrix mass="0.5" radius="${foothold_radius}" length="${foothold_height}"/>
-    </link>
-    <joint name="fb1_2base_link3" type="fixed">
-        <parent link="base_link_3"/>
-        <child link="foothold_base_1"/>
-        <origin xyz="0.0 0.0 0.0"/>
-    </joint>
-    <link name="foothold_base_2">
-        <visual>
-            <geometry>
-                <box size="${foothold_height} 0.05 0.23"/>
-            </geometry>
-            <material name="black" />
-        </visual>
-        <collision>
-            <geometry>
-                <box size="${foothold_height} 0.05 0.23"/>
-            </geometry>
-        </collision>
-        <xacro:box_inertial_matrix mass="0.1" length="${foothold_height}" width="0.05" height="0.23"/>
-    </link>
-    <joint name="foothold_base12_joint" type="fixed">
-        <parent link="foothold_base_1"/>
-        <child link="foothold_base_2"/>
-        <origin xyz="${-foothold_radius+0.001} 0.0 0.115"/>
-    </joint>
-    <link name="foothold_base_3">
-        <visual>
-            <geometry>
-                <box size="0.06 0.05 ${foothold_height}"/>
-            </geometry>
-            <material name="black" />
-        </visual>
-        <collision>
-            <geometry>
-                <box size="0.06 0.05 ${foothold_height}"/>
-            </geometry>
-        </collision>
-        <xacro:box_inertial_matrix mass="0.1" length="0.06" width="0.05" height="${foothold_height}"/>
-    </link>
-    <joint name="foothold_base23_joint" type="fixed">
-        <parent link="foothold_base_2"/>
-        <child link="foothold_base_3"/>
-        <origin xyz="0.03 0.0 0.115"/>
-    </joint>
-    <link name="foothold_base_4">
-        <visual>
-            <geometry>
-                <cylinder radius="0.07" length="${foothold_height}"/>
-            </geometry>
-            <material name="black" />
-        </visual>
-        <collision>
-            <geometry>
-                <cylinder radius="0.07" length="${foothold_height}"/>
-            </geometry>
-        </collision>
-        <xacro:cylinder_inertial_matrix mass="0.1" radius="0.07" length="${foothold_height}"/>
-    </link>
-    <joint name="foothold_base34_joint" type="fixed">
-        <parent link="foothold_base_3"/>
-        <child link="foothold_base_4"/>
-        <origin xyz="0.1 0.0 0.0"/>
-    </joint>
-    <link name="camera_link">
-        <visual>
-            <geometry>
-                <cylinder radius="0.02" length="0.07"/>
-            </geometry>
-            <material name="black" />
-        </visual>
-        <collision>
-            <geometry>
-                <cylinder radius="0.02" length="0.07"/>
-            </geometry>
-        </collision>
-        <xacro:cylinder_inertial_matrix mass="0.2" radius="0.02" length="0.007"/>
-    </link>
-    <joint name="camera_link2foothold4" type="fixed">
-        <parent link="foothold_base_4"/>
-        <child link="camera_link"/>
-        <origin xyz="0.0 0.0 -0.035"/>
-        <axis xyz="0.0 0.0 1"/>
-    </joint>
-    <link name="camera">
-        <visual>
-            <geometry>
-                <sphere radius="${camera_radius}"/>
-            </geometry>
-            <material name="white"/>
-        </visual>
-        <collision>
-            <geometry>
-                <sphere radius="${camera_radius}"/>
-            </geometry>
-        </collision>
-        <xacro:sphere_inertial_matrix mass="0.2" radius="${camera_radius}" />
-    </link>
-    <joint name="camera_link2camera" type="fixed">
-        <parent link="camera_link"/>
-        <child link="camera"/>
-        <origin xyz="0.0 0.0 ${-(camera_radius+0.035)}"/>
-    </joint>
+    <xacro:macro name="camera_func" params="parent *origin">
+        <link name="camera_base_footprint" />
+        <joint name="camera_base_joint" type="fixed">
+            <xacro:insert_block name="origin"/>
+            <parent link="${parent}"/>
+            <child link="camera_base_footprint"/>
+        </joint>
+        <link name="foothold_base_1">
+            <visual>
+                <geometry>
+                    <cylinder radius="${foothold_radius}" length="${foothold_height}"/>
+                </geometry>
+                <material name="black" />
+            </visual>
+            <collision>
+                <geometry>
+                    <cylinder radius="${foothold_radius}" length="${foothold_height}"/>
+                </geometry>
+            </collision>
+            <xacro:cylinder_inertial_matrix mass="0.5" radius="${foothold_radius}" length="${foothold_height}"/>
+        </link>
+        <joint name="fb1_2base_link3" type="fixed">
+            <parent link="camera_base_footprint"/>
+            <child link="foothold_base_1"/>
+            <origin xyz="0.0 0.0 ${foothold_height/2}"/>
+        </joint>
+        <link name="foothold_base_2">
+            <visual>
+                <geometry>
+                    <box size="${foothold_height} 0.05 0.23"/>
+                </geometry>
+                <material name="black" />
+            </visual>
+            <collision>
+                <geometry>
+                    <box size="${foothold_height} 0.05 0.23"/>
+                </geometry>
+            </collision>
+            <xacro:box_inertial_matrix mass="0.1" length="${foothold_height}" width="0.05" height="0.23"/>
+        </link>
+        <joint name="foothold_base12_joint" type="fixed">
+            <parent link="foothold_base_1"/>
+            <child link="foothold_base_2"/>
+            <origin xyz="${-foothold_radius+0.001} 0.0 0.115"/>
+        </joint>
+        <link name="foothold_base_3">
+            <visual>
+                <geometry>
+                    <box size="0.06 0.05 ${foothold_height}"/>
+                </geometry>
+                <material name="black" />
+            </visual>
+            <collision>
+                <geometry>
+                    <box size="0.06 0.05 ${foothold_height}"/>
+                </geometry>
+            </collision>
+            <xacro:box_inertial_matrix mass="0.1" length="0.06" width="0.05" height="${foothold_height}"/>
+        </link>
+        <joint name="foothold_base23_joint" type="fixed">
+            <parent link="foothold_base_2"/>
+            <child link="foothold_base_3"/>
+            <origin xyz="0.03 0.0 0.115"/>
+        </joint>
+        <link name="foothold_base_4">
+            <visual>
+                <geometry>
+                    <cylinder radius="0.07" length="${foothold_height}"/>
+                </geometry>
+                <material name="black" />
+            </visual>
+            <collision>
+                <geometry>
+                    <cylinder radius="0.07" length="${foothold_height}"/>
+                </geometry>
+            </collision>
+            <xacro:cylinder_inertial_matrix mass="0.1" radius="0.07" length="${foothold_height}"/>
+        </link>
+        <joint name="foothold_base34_joint" type="fixed">
+            <parent link="foothold_base_3"/>
+            <child link="foothold_base_4"/>
+            <origin xyz="0.1 0.0 0.0"/>
+        </joint>
+        <link name="camera_link">
+            <visual>
+                <geometry>
+                    <cylinder radius="0.02" length="0.07"/>
+                </geometry>
+                <material name="black" />
+            </visual>
+            <collision>
+                <geometry>
+                    <cylinder radius="0.02" length="0.07"/>
+                </geometry>
+            </collision>
+            <xacro:cylinder_inertial_matrix mass="0.2" radius="0.02" length="0.007"/>
+        </link>
+        <joint name="camera_link2foothold4" type="fixed">
+            <parent link="foothold_base_4"/>
+            <child link="camera_link"/>
+            <origin xyz="0.0 0.0 -0.035"/>
+            <axis xyz="0.0 0.0 1"/>
+        </joint>
+        <link name="camera">
+            <visual>
+                <geometry>
+                    <sphere radius="${camera_radius}"/>
+                </geometry>
+                <material name="white"/>
+            </visual>
+            <collision>
+                <geometry>
+                    <sphere radius="${camera_radius}"/>
+                </geometry>
+            </collision>
+            <xacro:sphere_inertial_matrix mass="0.2" radius="${camera_radius}" />
+        </link>
+        <joint name="camera_link2camera" type="fixed">
+            <parent link="camera_link"/>
+            <child link="camera"/>
+            <origin xyz="0.0 0.0 ${-(camera_radius+0.035)}"/>
+        </joint>
+    </xacro:macro>
 </robot>

File: src/bot_description/urdf/bot_gazebo_plugin.xacro (robot description, xacro)
@@ -16,8 +16,8 @@
 			<publishOdomTF>true</publishOdomTF>
 			<WheelTorque>30</WheelTorque>
-			<WheelSeparationW>0.35</WheelSeparationW>
-			<WheelSeparationL>0.6</WheelSeparationL>
+			<WheelSeparationW>0.36</WheelSeparationW>
+			<WheelSeparationL>0.32</WheelSeparationL>
 			<wheelAccel>10</wheelAccel>
-			<wheelDiameter>0.13</wheelDiameter>
+			<wheelDiameter>0.127</wheelDiameter>
 			<publishOdom>true</publishOdom>
 			<isRollerModel>true</isRollerModel>
