Commit message: feat:navigation

File: src/bot_description/urdf/bot_base.urdf.xacro (robot description, xacro)
@@ -32,6 +32,6 @@
     <xacro:property name="motor_mass" value="0.3" />
     <link name="base_footprint"/>
-    <!--   Define three chassis base_link_1 base_link_2 base_link_3-->
-    <link name="base_link_1">
+    <!--   Define three chassis base_link base_link_2 base_link_3-->
+    <link name="base_link">
         <visual>
             <geometry>
@@ -49,5 +49,5 @@
     <joint name="base_joint" type="fixed">
         <parent link="base_footprint"/>
-        <child link="base_link_1"/>
+        <child link="base_link"/>
         <origin xyz="0.0 0.0 ${z_offset+bot_height/2}"/>
     </joint>
@@ -81,5 +81,5 @@
     </link>
     <joint name="base12_joint" type="fixed">
-        <parent link="base_link_1"/>
+        <parent link="base_link"/>
         <child link="base_link_2"/>
         <origin xyz="0.0 0.0 ${pillar_height_1+bot_height}"/>
@@ -111,5 +111,5 @@
         </link>
         <joint name="${link_name}_joint" type="continuous">
-            <parent link="base_link_1"/>
+            <parent link="base_link"/>
             <child link="${link_name}"/>
             <origin xyz="${wheel_joint_x * front_flag} ${wheel_joint_y * left_flag} ${wheel_joint_z}"/>
@@ -119,5 +119,5 @@
         <xacro:mecanum_wheel name="${link_name}" roller_angle = "${angle*roller_angle}"/>
         <joint name="${link_name}_joint" type="continuous">
-            <parent link="base_link_1"/>
+            <parent link="base_link"/>
             <child link="${link_name}"/>
             <origin xyz="${wheel_joint_x * front_flag} ${wheel_joint_y * left_flag} ${wheel_joint_z}" rpy="${3*pi/2} 0 0"/>
@@ -154,5 +154,5 @@
         </link>
         <joint name="${link_name}_p1base_joint" type="fixed">
-            <parent link="base_link_1"/>
+            <parent link="base_link"/>
             <child link="${link_name}_p1"/>
             <origin xyz="${(bot_length/2-pillar_length/2) * front_flag} ${(bot_width/3) * left_flag} ${bot_height/2+pillar_height_1/2}"/>
@@ -181,5 +181,5 @@
         </link>
         <joint name="${link_name}_motor_joint" type="fixed">
-            <parent link="base_link_1"/>
+            <parent link="base_link"/>
             <child link="${link_name}_motor"/>
             <origin xyz="${wheel_joint_x * front_flag} ${((bot_width-motor_length)/2+wheel_base_dis) * left_flag} ${wheel_joint_z}"/>

File: src/bot_description/urdf/bot_gazebo.xacro (robot description, xacro)
@@ -3,6 +3,6 @@
     <xacro:include filename="$(find bot_description)/urdf/bot_roller.gazebo.xacro"/>
 	<xacro:include filename="$(find bot_description)/urdf/bot_roller.transmission.xacro"/>
-	<!-- base_link_1 gazebo -->
-	<gazebo reference="base_link_1">
+	<!-- base_link gazebo -->
+	<gazebo reference="base_link">
 		<selfCollide>false</selfCollide>
 		<gravity>true</gravity>

File: src/bot_description/urdf/bot_gazebo_plugin.xacro (robot description, xacro)
@@ -136,18 +136,30 @@
 			<horizontal_fov>1.047198</horizontal_fov>
 			<image>
-			<width>960</width>
-			<height>540</height>
-			<format>R8G8B8</format>
+				<width>960</width>
+				<height>540</height>
+				<format>R8G8B8</format>
 			</image>
 			<clip>
-			<near>0.05</near>
-			<far>3</far>
+				<near>0.05</near>
+				<far>3</far>
 			</clip>
 		</camera>
 		<plugin name="bot_depth_camera" filename="libgazebo_ros_camera.so">
-			<camera_name>camera</camera_name>
+			<baseline>0.2</baseline>
+			<alwaysOn>true</alwaysOn>
+			<updateRate>0.0</updateRate>
 			<frame_name>camera</frame_name>
-			<triggered>false</triggered>
-			<hack_baseline>0.07</hack_baseline>
+			<pointCloudCutoff>0.5</pointCloudCutoff>
+			<pointCloudCutoffMax>3.0</pointCloudCutoffMax>
+			<distortionK1>0</distortionK1>
+			<distortionK2>0</distortionK2>
+			<distortionK3>0</distortionK3>
+			<distortionT1>0</distortionT1>
+			<distortionT2>0</distortionT2>
+			<CxPrime>0</CxPrime>
+			<Cx>0</Cx>
+			<Cy>0</Cy>
+			<focalLength>0</focalLength>
+			<hackBaseline>0</hackBaseline>
 		</plugin>
 		</sensor>
